Commit message: set up inertial

File: urdf/kamuy2.urdf (robot description, URDF)
Before this commit: robot kamuy2, 17 links, 16 joints
Links:
- link back_left_link_first: mass 0.34395759179931723 -> 1.4
- link back_left_link_foot: mass 0.2932724386587248 -> 0.5
- link back_left_link_second: mass 0.08058045794484539 -> 0.5
- link back_right_link_first: mass 0.34395759179934193 -> 1.4
- link back_right_link_foot: mass 0.29327243865872493 -> 0.5
- link back_right_link_second: mass 0.08058045794484527 -> 0.5
- link base_link: mass 3.1908830685300313 -> 10
- link front_left_link_first: mass 0.34395759179934193 -> 1.4
- link front_left_link_foot: mass 0.2932724386587248 -> 0.5
- link front_left_link_second: mass 0.08058045794484539 -> 0.5
- link front_right_link_first: mass 0.34395759179931723 -> 1.4
- link front_right_link_foot: mass 0.29327243865872493 -> 0.5
- link front_right_link_second: mass 0.08058045794484527 -> 0.5
Joints:
- joint bl1: limit lower=-0.785398 upper=0.785398 effort=100 velocity=100 -> lower=-0.785398 upper=0.785398 effort=18 velocity=0.52
- joint bl2: limit lower=0.0 upper=3.141593 effort=100 velocity=100 -> lower=0.0 upper=3.141593 effort=18 velocity=0.52
- joint bl3: limit lower=0.0 upper=3.141593 effort=100 velocity=100 -> lower=0.0 upper=3.141593 effort=18 velocity=0.52
- joint bl4: limit lower=0.0 upper=3.141593 effort=100 velocity=100 -> lower=0.0 upper=3.141593 effort=18 velocity=0.52
- joint br1: limit lower=-0.785398 upper=0.785398 effort=100 velocity=100 -> lower=-0.785398 upper=0.785398 effort=18 velocity=0.52
- joint br2: limit lower=0.0 upper=3.141593 effort=100 velocity=100 -> lower=0.0 upper=3.141593 effort=18 velocity=0.52
- joint br3: limit lower=0.0 upper=3.141593 effort=100 velocity=100 -> lower=0.0 upper=3.141593 effort=18 velocity=0.52
- joint br4: limit lower=0.0 upper=3.141593 effort=100 velocity=100 -> lower=0.0 upper=3.141593 effort=18 velocity=0.52
- joint fl1: limit lower=-0.785398 upper=0.785398 effort=100 velocity=100 -> lower=-0.785398 upper=0.785398 effort=18 velocity=0.52
- joint fl2: limit lower=0.0 upper=3.141593 effort=100 velocity=100 -> lower=0.0 upper=3.141593 effort=18 velocity=0.52
- joint fl3: limit lower=0.0 upper=3.141593 effort=100 velocity=100 -> lower=0.0 upper=3.141593 effort=18 velocity=0.52
- joint fl4: limit lower=0.0 upper=3.141593 effort=100 velocity=100 -> lower=0.0 upper=3.141593 effort=18 velocity=0.52
- joint fr1: limit lower=-0.785398 upper=0.785398 effort=100 velocity=100 -> lower=-0.785398 upper=0.785398 effort=18 velocity=0.52
- joint fr2: limit lower=0.0 upper=3.141593 effort=100 velocity=100 -> lower=0.0 upper=3.141593 effort=18 velocity=0.52
- joint fr3: limit lower=0.0 upper=3.141593 effort=100 velocity=100 -> lower=0.0 upper=3.141593 effort=18 velocity=0.52
- joint fr4: limit lower=0.0 upper=3.141593 effort=100 velocity=100 -> lower=0.0 upper=3.141593 effort=18 velocity=0.52

File: urdf/kamuy2.xacro (robot description, xacro)
@@ -7,6 +7,6 @@
   <inertial>
     <origin xyz="0.00025193197119904756 0.0011290062234152254 0.10689635737270876" rpy="0 0 0"/>
-    <mass value="3.1908830685300313"/>
-    <inertia ixx="0.006226" iyy="0.123536" izz="0.126673" ixy="0.0" iyz="-7e-06" ixz="3e-06"/>
+    <mass value="10"/>
+    <inertia ixx="0.0666" iyy="0.24166" izz="0.24166" ixy="0.0" iyz="0" ixz="0"/>
   </inertial>
   <visual>
@@ -24,9 +24,10 @@
   </collision>
 </link>
+<!-- second link -->
 <link name="front_left_link_second">
   <inertial>
     <origin xyz="0 0 0" rpy="0 1.570796 0"/>
-    <mass value="0.08058045794484539"/>
-    <inertia ixx="0.000409" iyy="0.000392" izz="6.2e-05" ixy="0.0" iyz="4.8e-05" ixz="-0.0"/>
+    <mass value="0.5"/>
+    <inertia ixx="0.00712" iyy="0.007101" izz="0.000185416" ixy="0.0" iyz="0" ixz="0"/>
   </inertial>
   <visual>
@@ -47,6 +48,6 @@
   <inertial>
     <origin xyz="0 0 0" rpy="0 1.570796 0"/>
-    <mass value="0.08058045794484539"/>
-    <inertia ixx="0.000409" iyy="0.000392" izz="6.2e-05" ixy="0.0" iyz="4.8e-05" ixz="-0.0"/>
+    <mass value="0.5"/>
+    <inertia ixx="0.00712" iyy="0.007101" izz="0.000185416" ixy="0.0" iyz="0" ixz="0"/>
   </inertial>
   <visual>
@@ -67,6 +68,6 @@
   <inertial>
     <origin xyz="0 0 0" rpy="0 1.570796 0"/>
-    <mass value="0.08058045794484527"/>
-    <inertia ixx="0.000409" iyy="0.000392" izz="6.2e-05" ixy="-0.0" iyz="-4.8e-05" ixz="-0.0"/>
+    <mass value="0.5"/>
+    <inertia ixx="0.00712" iyy="0.007101" izz="0.000185416" ixy="0.0" iyz="0" ixz="0"/>
   </inertial>
   <visual>
@@ -87,6 +88,6 @@
   <inertial>
     <origin xyz="0 0 0" rpy="0 1.570796 0"/>
-    <mass value="0.08058045794484527"/>
-    <inertia ixx="0.000409" iyy="0.000392" izz="6.2e-05" ixy="-0.0" iyz="-4.8e-05" ixz="-0.0"/>
+    <mass value="0.5"/>
+    <inertia ixx="0.00712" iyy="0.007101" izz="0.000185416" ixy="0.0" iyz="0" ixz="0"/>
   </inertial>
   <visual>
@@ -104,9 +105,10 @@
   </collision>
 </link>
+<!-- first link -->
 <link name="front_right_link_first">
   <inertial>
     <origin xyz="0 0 0" rpy="0 0 0"/>
-    <mass value="0.34395759179931723"/>
-    <inertia ixx="0.000244" iyy="0.001214" izz="0.001272" ixy="-5e-05" iyz="1e-06" ixz="-4e-06"/>
+    <mass value="1.4"/>
+    <inertia ixx="0.001666" iyy="0.005413" izz="0.0050866" ixy="0" iyz="0" ixz="0"/>
   </inertial>
   <visual>
@@ -127,6 +129,6 @@
   <inertial>
     <origin xyz="0 0 0" rpy="0 0 0"/>
-    <mass value="0.34395759179934193"/>
-    <inertia ixx="0.000244" iyy="0.001214" izz="0.001272" ixy="5e-05" iyz="-1e-06" ixz="-4e-06"/>
+    <mass value="1.4"/>
+    <inertia ixx="0.001666" iyy="0.005413" izz="0.0050866" ixy="0" iyz="0" ixz="0"/>
   </inertial>
   <visual>
@@ -147,6 +149,6 @@
   <inertial>
     <origin xyz="0 0 0" rpy="0 0 0"/>
-    <mass value="0.34395759179934193"/>
-    <inertia ixx="0.000244" iyy="0.001214" izz="0.001272" ixy="5e-05" iyz="1e-06" ixz="4e-06"/>
+    <mass value="1.4"/>
+    <inertia ixx="0.001666" iyy="0.005413" izz="0.0050866" ixy="0" iyz="0" ixz="0"/>
   </inertial>
   <visual>
@@ -167,6 +169,6 @@
   <inertial>
     <origin xyz="0.0944653660519865 0.003464242618647702 -0.03287189320851288" rpy="0 0 0"/>
-    <mass value="0.34395759179931723"/>
-    <inertia ixx="0.000244" iyy="0.001214" izz="0.001272" ixy="-5e-05" iyz="-1e-06" ixz="4e-06"/>
+    <mass value="1.4"/>
+    <inertia ixx="0.001666" iyy="0.005413" izz="0.0050866" ixy="0" iyz="0" ixz="0"/>
   </inertial>
   <visual>
@@ -184,9 +186,10 @@
   </collision>
 </link>
+<!-- foot -->
 <link name="back_left_link_foot">
   <inertial>
     <origin xyz="0 0 0" rpy="0 1.570796 0"/>
-    <mass value="0.2932724386587248"/>
-    <inertia ixx="0.002288" iyy="0.002324" izz="0.00015" ixy="4e-06" iyz="1e-05" ixz="-0.000187"/>
+    <mass value="0.5"/>
+    <inertia ixx="0.00770833" iyy="0.00895833" izz="0.003333" ixy="0" iyz="0" ixz="-0.0025"/>
   </inertial>
   <visual>
@@ -207,6 +210,6 @@
   <inertial>
     <origin xyz="0 0 0" rpy="0 1.570796 0"/>
-    <mass value="0.2932724386587248"/>
-    <inertia ixx="0.002288" iyy="0.002324" izz="0.00015" ixy="4e-06" iyz="1e-05" ixz="-0.000187"/>
+    <mass value="0.5"/>
+   <inertia ixx="0.00770833" iyy="0.00895833" izz="0.003333" ixy="0" iyz="0" ixz="-0.0025"/>
   </inertial>
   <visual>
@@ -227,6 +230,6 @@
   <inertial>
     <origin xyz="0 0 0" rpy="3.141592 1.570796 0"/>
-    <mass value="0.29327243865872493"/>
-    <inertia ixx="0.002288" iyy="0.002324" izz="0.00015" ixy="-4e-06" iyz="-1e-05" ixz="-0.000187"/>
+    <mass value="0.5"/>
+    <inertia ixx="0.00770833" iyy="0.00895833" izz="0.003333" ixy="0" iyz="0" ixz="-0.0025"/>
   </inertial>
   <visual>
@@ -247,6 +250,6 @@
   <inertial>
     <origin xyz="0 0 0" rpy="3.141592 1.570796 0"/>
-    <mass value="0.29327243865872493"/>
-    <inertia ixx="0.002288" iyy="0.002324" izz="0.00015" ixy="-4e-06" iyz="-1e-05" ixz="-0.000187"/>
+    <mass value="0.5"/>
+   <inertia ixx="0.00770833" iyy="0.00895833" izz="0.003333" ixy="0" iyz="0" ixz="-0.0025"/>
   </inertial>
   <visual>
@@ -278,5 +281,5 @@
   <child link="front_right_link_first"/>
   <axis xyz="-1.0 0.0 0.0"/>
-  <limit upper="0.785398" lower="-0.785398" effort="100" velocity="100"/>
+  <limit upper="0.785398" lower="-0.785398" effort="18" velocity="0.52"/>
 </joint>
 <joint name="fl1" type="revolute">
@@ -285,5 +288,5 @@
   <child link="front_left_link_first"/>
   <axis xyz="-1.0 0.0 0.0"/>
-  <limit upper="0.785398" lower="-0.785398" effort="100" velocity="100"/>
+  <limit upper="0.785398" lower="-0.785398" effort="18" velocity="0.52"/>
 </joint>
 <joint name="br1" type="revolute">
@@ -292,5 +295,5 @@
   <child link="back_right_link_first"/>
   <axis xyz="-1.0 5e-06 -0.0"/>
-  <limit upper="0.785398" lower="-0.785398" effort="100" velocity="100"/>
+  <limit upper="0.785398" lower="-0.785398" effort="18" velocity="0.52"/>
 </joint>
 <joint name="bl1" type="revolute">
@@ -299,5 +302,5 @@
   <child link="back_left_link_first"/>
   <axis xyz="-1.0 5e-06 -0.0"/>
-  <limit upper="0.785398" lower="-0.785398" effort="100" velocity="100"/>
+  <limit upper="0.785398" lower="-0.785398" effort="18" velocity="0.52"/>
 </joint>
 <joint name="fl2" type="revolute">
@@ -306,5 +309,5 @@
   <child link="front_left_link_second"/>
   <axis xyz="0.0 1.0 0.0"/>
-  <limit upper="3.141593" lower="0.0" effort="100" velocity="100"/>
+  <limit upper="3.141593" lower="0.0" effort="18" velocity="0.52"/>
 </joint>
 <joint name="bl2" type="revolute">
@@ -313,5 +316,5 @@
   <child link="back_left_link_second"/>
   <axis xyz="-5e-06 -1.0 -0.0"/>
-  <limit upper="0.087266" lower="-3.141593" effort="100" velocity="100"/>
+  <limit upper="0.087266" lower="-3.141593" effort="18" velocity="0.52"/>
 </joint>
 <joint name="fr2" type="revolute">
@@ -320,5 +323,5 @@
   <child link="front_right_link_second"/>
   <axis xyz="-0.0 1.0 -0.0"/>
-  <limit upper="3.141593" lower="0.0" effort="100" velocity="100"/>
+  <limit upper="3.141593" lower="0.0" effort="18" velocity="0.52"/>
 </joint>
 <joint name="br2" type="revolute">
@@ -327,5 +330,5 @@
   <child link="back_right_link_second"/>
   <axis xyz="-5e-06 -1.0 -0.0"/>
-  <limit upper="0.0" lower="-3.141593" effort="100" velocity="100"/>
+  <limit upper="0.0" lower="-3.141593" effort="18" velocity="0.52"/>
 </joint>
 <joint name="bl3" type="revolute">
@@ -334,5 +337,5 @@
   <child link="back_left_link_foot"/>
   <axis xyz="-5e-06 -1.0 -0.0"/>
-  <limit upper="3.141593" lower="0.0" effort="100" velocity="100"/>
+  <limit upper="3.141593" lower="0.0" effort="18" velocity="0.52"/>
 </joint>
 <joint name="fl3" type="revolute">
@@ -341,5 +344,5 @@
   <child link="front_left_link_foot"/>
   <axis xyz="-0.0 -1.0 -0.0"/>
-  <limit upper="3.141593" lower="0.0" effort="100" velocity="100"/>
+  <limit upper="3.141593" lower="0.0" effort="18" velocity="0.52"/>
 </joint>
 <joint name="fr3" type="revolute">
@@ -348,5 +351,5 @@
   <child link="front_right_link_foot"/>
   <axis xyz="0.0 -1.0 0.0"/>
-  <limit upper="3.141593" lower="0.0" effort="100" velocity="100"/>
+  <limit upper="3.141593" lower="0.0" effort="18" velocity="0.52"/>
 </joint>
 <joint name="br3" type="revolute">
@@ -355,5 +358,5 @@
   <child link="back_right_link_foot"/>
   <axis xyz="-5e-06 -1.0 -0.0"/>
-  <limit upper="3.141593" lower="0.0" effort="100" velocity="100"/>
+  <limit upper="3.141593" lower="0.0" effort="18" velocity="0.52"/>
 </joint>
 -->
@@ -363,5 +366,5 @@
   <child link="front_right_link_first"/>
   <axis xyz="-1.0 0.0 0.0"/>
-  <limit upper="0.785398" lower="-0.785398" effort="100" velocity="100"/>
+  <limit upper="0.785398" lower="-0.785398" effort="18" velocity="0.52"/>
 </joint>
 <joint name="fl1" type="revolute">
@@ -370,5 +373,5 @@
   <child link="front_left_link_first"/>
   <axis xyz="-1.0 0.0 0.0"/>
-  <limit upper="0.785398" lower="-0.785398" effort="100" velocity="100"/>
+  <limit upper="0.785398" lower="-0.785398" effort="18" velocity="0.52"/>
 </joint>
 <joint name="br1" type="revolute">
@@ -377,5 +380,5 @@
   <child link="back_right_link_first"/>
   <axis xyz="-1.0 5e-06 -0.0"/>
-  <limit upper="0.785398" lower="-0.785398" effort="100" velocity="100"/>
+  <limit upper="0.785398" lower="-0.785398" effort="18" velocity="0.52"/>
 </joint>
 <joint name="bl1" type="revolute">
@@ -384,5 +387,5 @@
   <child link="back_left_link_first"/>
   <axis xyz="-1.0 5e-06 -0.0"/>
-  <limit upper="0.785398" lower="-0.785398" effort="100" velocity="100"/>
+  <limit upper="0.785398" lower="-0.785398" effort="18" velocity="0.52"/>
 </joint>
 <joint name="fl2" type="revolute">
@@ -391,5 +394,5 @@
   <child link="front_left_link_second"/>
   <axis xyz="0.0 1.0 0.0"/>
-  <limit upper="3.141593" lower="0.0" effort="100" velocity="100"/>
+  <limit upper="3.141593" lower="0.0" effort="18" velocity="0.52"/>
 </joint>
 <joint name="bl2" type="revolute">
@@ -398,5 +401,5 @@
   <child link="back_left_link_second"/>
   <axis xyz="0.0 1.0 0.0"/>
-  <limit upper="3.141593" lower="0.0" effort="100" velocity="100"/>
+  <limit upper="3.141593" lower="0.0" effort="18" velocity="0.52"/>
 </joint>
 <joint name="fr2" type="revolute">
@@ -405,5 +408,5 @@
   <child link="front_right_link_second"/>
   <axis xyz="-0.0 1.0 -0.0"/>
-  <limit upper="3.141593" lower="0.0" effort="100" velocity="100"/>
+  <limit upper="3.141593" lower="0.0" effort="18" velocity="0.52"/>
 </joint>
 <joint name="br2" type="revolute">
@@ -412,5 +415,5 @@
   <child link="back_right_link_second"/>
   <axis xyz="-0.0 1.0 -0.0"/>
-  <limit upper="3.141593" lower="0.0" effort="100" velocity="100"/>
+  <limit upper="3.141593" lower="0.0" effort="18" velocity="0.52"/>
 </joint>
 <joint name="bl3" type="revolute">
@@ -419,5 +422,5 @@
   <child link="back_left_link_foot"/>
   <axis xyz="0 1 -0.0"/>
-  <limit upper="3.141593" lower="0.0" effort="100" velocity="100"/>
+  <limit upper="3.141593" lower="0.0" effort="18" velocity="0.52"/>
 </joint>
 <joint name="fl3" type="revolute">
@@ -426,5 +429,5 @@
   <child link="front_left_link_foot"/>
   <axis xyz="-0.0 1.0 -0.0"/>
-  <limit upper="3.141593" lower="0.0" effort="100" velocity="100"/>
+  <limit upper="3.141593" lower="0.0" effort="18" velocity="0.52"/>
 </joint>
 <joint name="fr3" type="revolute">
@@ -433,5 +436,5 @@
   <child link="front_right_link_foot"/>
   <axis xyz="0.0 1.0 0.0"/>
-  <limit upper="3.141593" lower="0.0" effort="100" velocity="100"/>
+  <limit upper="3.141593" lower="0.0" effort="18" velocity="0.52"/>
 </joint>
 <joint name="br3" type="revolute">
@@ -440,5 +443,5 @@
   <child link="back_right_link_foot"/>
   <axis xyz="0 1.0 -0.0"/>
-  <limit upper="3.141593" lower="0.0" effort="100" velocity="100"/>
+  <limit upper="3.141593" lower="0.0" effort="18" velocity="0.52"/>
 </joint>
 <joint name="fl4" type="fixed">
@@ -447,5 +450,5 @@
   <child link="front_left_foot"/>
   <axis xyz="0.0 1.0 -0.0"/>
-  <limit upper="3.141593" lower="0.0" effort="100" velocity="100"/>
+  <limit upper="3.141593" lower="0.0" effort="18" velocity="0.52"/>
 </joint>
 <joint name="fr4" type="fixed">
@@ -454,5 +457,5 @@
   <child link="front_right_foot"/>
   <axis xyz="0.0 1.0 -0.0"/>
-  <limit upper="3.141593" lower="0.0" effort="100" velocity="100"/>
+  <limit upper="3.141593" lower="0.0" effort="18" velocity="0.52"/>
 </joint>
 <joint name="bl4" type="fixed">
@@ -461,5 +464,5 @@
   <child link="back_left_foot"/>
   <axis xyz="0.0 1.0 -0.0"/>
-  <limit upper="3.141593" lower="0.0" effort="100" velocity="100"/>
+  <limit upper="3.141593" lower="0.0" effort="18" velocity="0.52"/>
 </joint>
 <joint name="br4" type="fixed">
@@ -468,5 +471,5 @@
   <child link="back_right_foot"/>
   <axis xyz="-0.0 -1.0 -0.0"/>
-  <limit upper="3.141593" lower="0.0" effort="100" velocity="100"/>
+  <limit upper="3.141593" lower="0.0" effort="18" velocity="0.52"/>
 </joint>
 </robot>
