Commit message: change to adapt to gazebo

File: urdf/kamuy2.urdf (robot description, URDF)
Before this commit: robot kamuy2, 17 links, 16 joints
Links:
- link back_left_foot: geometry collision sphere radius=0.03; visual sphere radius=0.03
- link back_right_foot: geometry collision sphere radius=0.03; visual sphere radius=0.03
- link front_left_foot: geometry collision sphere radius=0.03; visual sphere radius=0.03
- link front_right_foot: geometry collision sphere radius=0.03; visual sphere radius=0.03
Joints:
- joint bl3: limit lower=0.0 upper=3.141593 effort=18 velocity=0.52 -> lower=-3.141592 upper=0 effort=18 velocity=0.52
- joint br3: limit lower=0.0 upper=3.141593 effort=18 velocity=0.52 -> lower=-3.141592 upper=0 effort=18 velocity=0.52
- joint fl3: limit lower=0.0 upper=3.141593 effort=18 velocity=0.52 -> lower=-3.141592 upper=0 effort=18 velocity=0.52
- joint fr3: limit lower=0.0 upper=3.141593 effort=18 velocity=0.52 -> lower=-3.141592 upper=0 effort=18 velocity=0.52

File: urdf/kamuy2.xacro (robot description, xacro)
@@ -6,10 +6,10 @@
 <link name="base_link">
   <inertial>
-    <origin xyz="0.00025193197119904756 0.0011290062234152254 0.10689635737270876" rpy="0 0 0"/>
-    <mass value="10"/>
+    <origin xyz="0 -0.01 0.03" rpy="0 0 0"/>
+    <mass value="5"/>
     <inertia ixx="0.0666" iyy="0.24166" izz="0.24166" ixy="0.0" iyz="0" ixz="0"/>
   </inertial>
   <visual>
-    <origin xyz="0 0 0.03" rpy="0 0 0"/>
+    <origin xyz="0 -0.01 0.03" rpy="0 0 0"/>
     <geometry>
       <mesh filename="package://kamuy2_description/meshes/base_link.stl" scale="0.001 0.001 0.001"/>
@@ -18,9 +18,45 @@
   </visual>
   <collision>
-    <origin xyz="0 0 0.03" rpy="0 0 0"/>
+    <origin xyz="0 -0.01 0.03" rpy="0 0 0"/>
     <geometry>
       <mesh filename="package://kamuy2_description/meshes/base_link.stl" scale="0.001 0.001 0.001"/>
     </geometry>
-  </collision>
+                          <surface>
+                    <friction>
+                        <ode>
+                            <mu>10</mu>
+                            <mu2>10</mu2>
+                        </ode>
+                    </friction>
+                </surface>
+  </collision>
+</link>
+<!-- sensor -->
+<link name="camera_link">
+  <visual>
+    <origin xyz="0 0.0 0" rpy="0 0 0"/>
+    <geometry>
+      <sphere radius="0.05"/>
+    </geometry>
+    <material name="silver"/>
+  </visual>
+</link>
+<link name="imu_link">
+  <visual>
+    <origin xyz="0 0.0 0" rpy="0 0 0"/>
+    <geometry>
+      <sphere radius="0.05"/>
+    </geometry>
+    <material name="silver"/>
+  </visual>
+</link>
+<link name="lidar_link">
+  <visual>
+    <origin xyz="0 0.0 0" rpy="0 0 0"/>
+    <geometry>
+      <sphere radius="0.05"/>
+    </geometry>
+    <material name="silver"/>
+  </visual>
 </link>
 <!-- second link -->
@@ -43,4 +79,12 @@
       <mesh filename="package://kamuy2_description/meshes/front_left_link_second.stl" scale="0.001 0.001 0.001"/>
     </geometry>
+                          <surface>
+                    <friction>
+                        <ode>
+                            <mu>10</mu>
+                            <mu2>10</mu2>
+                        </ode>
+                    </friction>
+                </surface>
   </collision>
 </link>
@@ -63,4 +107,12 @@
       <mesh filename="package://kamuy2_description/meshes/back_left_link_second.stl" scale="0.001 0.001 0.001"/>
     </geometry>
+                          <surface>
+                    <friction>
+                        <ode>
+                            <mu>10</mu>
+                            <mu2>10</mu2>
+                        </ode>
+                    </friction>
+                </surface>
   </collision>
 </link>
@@ -83,4 +135,12 @@
       <mesh filename="package://kamuy2_description/meshes/front_right_link_second.stl" scale="0.001 0.001 0.001"/>
     </geometry>
+                          <surface>
+                    <friction>
+                        <ode>
+                            <mu>10</mu>
+                            <mu2>10</mu2>
+                        </ode>
+                    </friction>
+                </surface>
   </collision>
 </link>
@@ -103,4 +163,12 @@
       <mesh filename="package://kamuy2_description/meshes/back_right_link_second.stl" scale="0.001 0.001 0.001"/>
     </geometry>
+                          <surface>
+                    <friction>
+                        <ode>
+                            <mu>10</mu>
+                            <mu2>10</mu2>
+                        </ode>
+                    </friction>
+                </surface>
   </collision>
 </link>
@@ -113,5 +181,5 @@
   </inertial>
   <visual>
-    <origin xyz="0 0 0" rpy="0 0 0"/>
+    <origin xyz="0 0 0" rpy="0 0 3.141592"/>
     <geometry>
       <mesh filename="package://kamuy2_description/meshes/front_right_link_first.stl" scale="0.001 0.001 0.001"/>
@@ -120,8 +188,16 @@
   </visual>
   <collision>
-    <origin xyz="0 0 0" rpy="0 0 0"/>
+    <origin xyz="0 0 0" rpy="0 0 3.141592"/>
     <geometry>
       <mesh filename="package://kamuy2_description/meshes/front_right_link_first.stl" scale="0.001 0.001 0.001"/>
     </geometry>
+                          <surface>
+                    <friction>
+                        <ode>
+                            <mu>10</mu>
+                            <mu2>10</mu2>
+                        </ode>
+                    </friction>
+                </surface>
   </collision>
 </link>
@@ -133,5 +209,5 @@
   </inertial>
   <visual>
-    <origin xyz="0 0 0" rpy="0 0 0"/>
+    <origin xyz="0 0 0" rpy="0 0 3.141592"/>
     <geometry>
       <mesh filename="package://kamuy2_description/meshes/front_left_link_first.stl" scale="0.001 0.001 0.001"/>
@@ -140,8 +216,16 @@
   </visual>
   <collision>
-    <origin xyz="0 0 0" rpy="0 0 0"/>
+    <origin xyz="0 0 0" rpy="0 0 3.141592"/>
     <geometry>
       <mesh filename="package://kamuy2_description/meshes/front_left_link_first.stl" scale="0.001 0.001 0.001"/>
     </geometry>
+                          <surface>
+                    <friction>
+                        <ode>
+                            <mu>10</mu>
+                            <mu2>10</mu2>
+                        </ode>
+                    </friction>
+                </surface>
   </collision>
 </link>
@@ -164,4 +248,12 @@
       <mesh filename="package://kamuy2_description/meshes/back_right_link_first.stl" scale="0.001 0.001 0.001"/>
     </geometry>
+                          <surface>
+                    <friction>
+                        <ode>
+                            <mu>10</mu>
+                            <mu2>10</mu2>
+                        </ode>
+                    </friction>
+                </surface>
   </collision>
 </link>
@@ -184,4 +276,12 @@
       <mesh filename="package://kamuy2_description/meshes/back_left_link_first.stl" scale="0.001 0.001 0.001"/>
     </geometry>
+                          <surface>
+                    <friction>
+                        <ode>
+                            <mu>10</mu>
+                            <mu2>10</mu2>
+                        </ode>
+                    </friction>
+                </surface>
   </collision>
 </link>
@@ -205,4 +305,12 @@
       <mesh filename="package://kamuy2_description/meshes/back_left_link_foot.stl" scale="0.001 0.001 0.001"/>
     </geometry>
+                    <surface>
+                    <friction>
+                        <ode>
+                            <mu>10</mu>
+                            <mu2>10</mu2>
+                        </ode>
+                    </friction>
+                </surface>
   </collision>
 </link>
@@ -225,4 +333,12 @@
       <mesh filename="package://kamuy2_description/meshes/front_left_link_foot.stl" scale="0.001 0.001 0.001"/>
     </geometry>
+                    <surface>
+                    <friction>
+                        <ode>
+                            <mu>10</mu>
+                            <mu2>10</mu2>
+                        </ode>
+                    </friction>
+                </surface>
   </collision>
 </link>
@@ -245,5 +361,13 @@
       <mesh filename="package://kamuy2_description/meshes/front_right_link_foot.stl" scale="0.001 0.001 0.001"/>
     </geometry>
-  </collision>
+                    <surface>
+                    <friction>
+                        <ode>
+                            <mu>10</mu>
+                            <mu2>10</mu2>
+                        </ode>
+                    </friction>
+                </surface>
+ </collision>
 </link>
 <link name="back_right_link_foot">
@@ -265,13 +389,113 @@
       <mesh filename="package://kamuy2_description/meshes/back_right_link_foot.stl" scale="0.001 0.001 0.001"/>
     </geometry>
+                    <surface>
+                    <friction>
+                        <ode>
+                            <mu>10</mu>
+                            <mu2>10</mu2>
+                        </ode>
+                    </friction>
+                </surface>
   </collision>
 </link>
 <link name="front_left_foot">
+  <inertial>
+    <origin xyz="0 0 0" rpy="0 0 0"/>
+    <mass value="0.1"/>
+    <inertia ixx="0.1" iyy="0.1" izz="0.1" ixy="0" iyz="0" ixz="0"/>
+  </inertial>
+    <visual>
+      <geometry>
+          <sphere radius="0.04"/>
+      </geometry>
+    </visual>
+    <collision>
+      <geometry>
+          <sphere radius="0.04"/>
+      </geometry>
+                <surface>
+                    <friction>
+                        <ode>
+                            <mu>10</mu>
+                            <mu2>10</mu2>
+                        </ode>
+                    </friction>
+                </surface>
+    </collision>
 </link>
 <link name="front_right_foot">
+  <inertial>
+    <origin xyz="0 0 0" rpy="0 0 0"/>
+    <mass value="0.1"/>
+    <inertia ixx="0.1" iyy="0.1" izz="0.1" ixy="0" iyz="0" ixz="0"/>
+  </inertial>
+    <visual>
+      <geometry>
+          <sphere radius="0.04"/>
+      </geometry>
+    </visual>
+    <collision>
+      <geometry>
+          <sphere radius="0.04"/>
+      </geometry>
+                      <surface>
+                    <friction>
+                        <ode>
+                            <mu>10</mu>
+                            <mu2>10</mu2>
+                        </ode>
+                    </friction>
+                </surface>
+    </collision>
 </link>
 <link name="back_left_foot">
+  <inertial>
+    <origin xyz="0 0 0" rpy="0 0 0"/>
+    <mass value="0.1"/>
+    <inertia ixx="0.1" iyy="0.1" izz="0.1" ixy="0" iyz="0" ixz="0"/>
+  </inertial>
+    <visual>
+      <geometry>
+          <sphere radius="0.04"/>
+      </geometry>
+    </visual>
+    <collision>
+      <geometry>
+          <sphere radius="0.04"/>
+      </geometry>
+                      <surface>
+                    <friction>
+                        <ode>
+                            <mu>10</mu>
+                            <mu2>10</mu2>
+                        </ode>
+                    </friction>
+                </surface>
+    </collision>
 </link>
 <link name="back_right_foot">
+  <inertial>
+    <origin xyz="0 0 0" rpy="0 0 0"/>
+    <mass value="0.1"/>
+    <inertia ixx="0.1" iyy="0.1" izz="0.1" ixy="0" iyz="0" ixz="0"/>
+  </inertial>
+    <visual>
+      <geometry>
+          <sphere radius="0.04"/>
+      </geometry>
+    </visual>
+    <collision>
+      <geometry>
+          <sphere radius="0.04"/>
+      </geometry>
+                      <surface>
+                    <friction>
+                        <ode>
+                            <mu>10</mu>
+                            <mu2>10</mu2>
+                        </ode>
+                    </friction>
+                </surface>
+    </collision>
 </link>
 <!--
@@ -281,5 +505,5 @@
   <child link="front_right_link_first"/>
   <axis xyz="-1.0 0.0 0.0"/>
-  <limit upper="0.785398" lower="-0.785398" effort="18" velocity="0.52"/>
+  <limit upper="0.785398" lower="-0.785398" effort="20" velocity="1.5"/>
 </joint>
 <joint name="fl1" type="revolute">
@@ -288,5 +512,5 @@
   <child link="front_left_link_first"/>
   <axis xyz="-1.0 0.0 0.0"/>
-  <limit upper="0.785398" lower="-0.785398" effort="18" velocity="0.52"/>
+  <limit upper="0.785398" lower="-0.785398" effort="20" velocity="1.5"/>
 </joint>
 <joint name="br1" type="revolute">
@@ -294,6 +518,6 @@
   <parent link="base_link"/>
   <child link="back_right_link_first"/>
-  <axis xyz="-1.0 5e-06 -0.0"/>
-  <limit upper="0.785398" lower="-0.785398" effort="18" velocity="0.52"/>
+  <axis xyz="-1.0 0 -0.0"/>
+  <limit upper="0.785398" lower="-0.785398" effort="20" velocity="1.5"/>
 </joint>
 <joint name="bl1" type="revolute">
@@ -301,6 +525,6 @@
   <parent link="base_link"/>
   <child link="back_left_link_first"/>
-  <axis xyz="-1.0 5e-06 -0.0"/>
-  <limit upper="0.785398" lower="-0.785398" effort="18" velocity="0.52"/>
+  <axis xyz="-1.0 0 -0.0"/>
+  <limit upper="0.785398" lower="-0.785398" effort="20" velocity="1.5"/>
 </joint>
 <joint name="fl2" type="revolute">
@@ -309,5 +533,5 @@
   <child link="front_left_link_second"/>
   <axis xyz="0.0 1.0 0.0"/>
-  <limit upper="3.141593" lower="0.0" effort="18" velocity="0.52"/>
+  <limit upper="3.141593" lower="0.0" effort="20" velocity="1.5"/>
 </joint>
 <joint name="bl2" type="revolute">
@@ -315,6 +539,6 @@
   <parent link="back_left_link_first"/>
   <child link="back_left_link_second"/>
-  <axis xyz="-5e-06 -1.0 -0.0"/>
-  <limit upper="0.087266" lower="-3.141593" effort="18" velocity="0.52"/>
+  <axis xyz="-0 -1.0 -0.0"/>
+  <limit upper="0.087266" lower="-3.141593" effort="20" velocity="1.5"/>
 </joint>
 <joint name="fr2" type="revolute">
@@ -323,12 +547,12 @@
   <child link="front_right_link_second"/>
   <axis xyz="-0.0 1.0 -0.0"/>
-  <limit upper="3.141593" lower="0.0" effort="18" velocity="0.52"/>
+  <limit upper="3.141593" lower="0.0" effort="20" velocity="1.5"/>
 </joint>
 <joint name="br2" type="revolute">
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