Commit message: モデルの向きを修正した

File: urdf/kamuy2.xacro (robot description, xacro)
@@ -226,10 +226,10 @@
 <link name="front_right_link_foot">
   <inertial>
-    <origin xyz="0 0 0" rpy="0 0 0"/>
+    <origin xyz="0 0 0" rpy="3.141592 0 0"/>
     <mass value="0.29327243865872493"/>
     <inertia ixx="0.002288" iyy="0.002324" izz="0.00015" ixy="-4e-06" iyz="-1e-05" ixz="-0.000187"/>
   </inertial>
   <visual>
-    <origin xyz="0 0 0" rpy="0 0 0"/>
+    <origin xyz="0 0 0" rpy="3.141592 0 0"/>
     <geometry>
       <mesh filename="package://kamuy2_description/meshes/front_right_link_foot.stl" scale="0.001 0.001 0.001"/>
@@ -238,5 +238,5 @@
   </visual>
   <collision>
-    <origin xyz="0 0 0" rpy="0 0 0"/>
+    <origin xyz="0 0 0" rpy="3.141592 0 0"/>
     <geometry>
       <mesh filename="package://kamuy2_description/meshes/front_right_link_foot.stl" scale="0.001 0.001 0.001"/>
@@ -246,10 +246,10 @@
 <link name="back_right_link_foot">
   <inertial>
-    <origin xyz="0 0 0" rpy="0 0 0"/>
+    <origin xyz="0 0 0" rpy="3.141592 0 0"/>
     <mass value="0.29327243865872493"/>
     <inertia ixx="0.002288" iyy="0.002324" izz="0.00015" ixy="-4e-06" iyz="-1e-05" ixz="-0.000187"/>
   </inertial>
   <visual>
-    <origin xyz="0 0 0" rpy="0 0 0"/>
+    <origin xyz="0 0 0" rpy="3.141592 0 0"/>
     <geometry>
       <mesh filename="package://kamuy2_description/meshes/back_right_link_foot.stl" scale="0.001 0.001 0.001"/>
@@ -258,5 +258,5 @@
   </visual>
   <collision>
-    <origin xyz="0 0 0" rpy="0 0 0"/>
+    <origin xyz="0 0 0" rpy="3.141592 0 0"/>
     <geometry>
       <mesh filename="package://kamuy2_description/meshes/back_right_link_foot.stl" scale="0.001 0.001 0.001"/>

Commit message: urdf調整

File: urdf/kamuy2.xacro (robot description, xacro)
@@ -26,10 +26,10 @@
 <link name="front_left_link_second">
   <inertial>
-    <origin xyz="0 0 0" rpy="0 0 0"/>
+    <origin xyz="0 0 0" rpy="0 1.570796 0"/>
     <mass value="0.08058045794484539"/>
     <inertia ixx="0.000409" iyy="0.000392" izz="6.2e-05" ixy="0.0" iyz="4.8e-05" ixz="-0.0"/>
   </inertial>
   <visual>
-    <origin xyz="0 0 0" rpy="0 0 0"/>
+    <origin xyz="0 0 0" rpy="0 1.570796 0"/>
     <geometry>
       <mesh filename="package://kamuy2_description/meshes/front_left_link_second.stl" scale="0.001 0.001 0.001"/>
@@ -38,5 +38,5 @@
   </visual>
   <collision>
-    <origin xyz="0 0 0" rpy="0 0 0"/>
+    <origin xyz="0 0 0" rpy="0 1.570796 0"/>
     <geometry>
       <mesh filename="package://kamuy2_description/meshes/front_left_link_second.stl" scale="0.001 0.001 0.001"/>
@@ -46,10 +46,10 @@
 <link name="back_left_link_second">
   <inertial>
-    <origin xyz="0 0 0" rpy="0 0 0"/>
+    <origin xyz="0 0 0" rpy="0 1.570796 0"/>
     <mass value="0.08058045794484539"/>
     <inertia ixx="0.000409" iyy="0.000392" izz="6.2e-05" ixy="0.0" iyz="4.8e-05" ixz="-0.0"/>
   </inertial>
   <visual>
-    <origin xyz="0 0 0" rpy="0 0 0"/>
+    <origin xyz="0 0 0" rpy="0 1.570796 0"/>
     <geometry>
       <mesh filename="package://kamuy2_description/meshes/back_left_link_second.stl" scale="0.001 0.001 0.001"/>
@@ -58,5 +58,5 @@
   </visual>
   <collision>
-    <origin xyz="0 0 0" rpy="0 0 0"/>
+    <origin xyz="0 0 0" rpy="0 1.570796 0"/>
     <geometry>
       <mesh filename="package://kamuy2_description/meshes/back_left_link_second.stl" scale="0.001 0.001 0.001"/>
@@ -66,10 +66,10 @@
 <link name="front_right_link_second">
   <inertial>
-    <origin xyz="0 0 0" rpy="0 0 0"/>
+    <origin xyz="0 0 0" rpy="0 1.570796 0"/>
     <mass value="0.08058045794484527"/>
     <inertia ixx="0.000409" iyy="0.000392" izz="6.2e-05" ixy="-0.0" iyz="-4.8e-05" ixz="-0.0"/>
   </inertial>
   <visual>
-    <origin xyz="0 0 0" rpy="0 0 0"/>
+    <origin xyz="0 0 0" rpy="0 1.570796 0"/>
     <geometry>
       <mesh filename="package://kamuy2_description/meshes/front_right_link_second.stl" scale="0.001 0.001 0.001"/>
@@ -78,5 +78,5 @@
   </visual>
   <collision>
-    <origin xyz="0 0 0" rpy="0 0 0"/>
+    <origin xyz="0 0 0" rpy="0 1.570796 0"/>
     <geometry>
       <mesh filename="package://kamuy2_description/meshes/front_right_link_second.stl" scale="0.001 0.001 0.001"/>
@@ -86,10 +86,10 @@
 <link name="back_right_link_second">
   <inertial>
-    <origin xyz="0 0 0" rpy="0 0 0"/>
+    <origin xyz="0 0 0" rpy="0 1.570796 0"/>
     <mass value="0.08058045794484527"/>
     <inertia ixx="0.000409" iyy="0.000392" izz="6.2e-05" ixy="-0.0" iyz="-4.8e-05" ixz="-0.0"/>
   </inertial>
   <visual>
-    <origin xyz="0 0 0" rpy="0 0 0"/>
+    <origin xyz="0 0 0" rpy="0 1.570796 0"/>
     <geometry>
       <mesh filename="package://kamuy2_description/meshes/back_right_link_second.stl" scale="0.001 0.001 0.001"/>
@@ -98,5 +98,5 @@
   </visual>
   <collision>
-    <origin xyz="0 0 0" rpy="0 0 0"/>
+    <origin xyz="0 0 0" rpy="0 1.570796 0"/>
     <geometry>
       <mesh filename="package://kamuy2_description/meshes/back_right_link_second.stl" scale="0.001 0.001 0.001"/>
@@ -186,10 +186,10 @@
 <link name="back_left_link_foot">
   <inertial>
-    <origin xyz="0 0 0" rpy="0 0 0"/>
+    <origin xyz="0 0 0" rpy="0 1.570796 0"/>
     <mass value="0.2932724386587248"/>
     <inertia ixx="0.002288" iyy="0.002324" izz="0.00015" ixy="4e-06" iyz="1e-05" ixz="-0.000187"/>
   </inertial>
   <visual>
-    <origin xyz="0 0 0" rpy="0 0 0"/>
+    <origin xyz="0 0 0" rpy="0 1.570796 0"/>
     <geometry>
       <mesh filename="package://kamuy2_description/meshes/back_left_link_foot.stl" scale="0.001 0.001 0.001"/>
@@ -198,5 +198,5 @@
   </visual>
   <collision>
-    <origin xyz="0 0 0" rpy="0 0 0"/>
+    <origin xyz="0 0 0" rpy="0 1.570796 0"/>
     <geometry>
       <mesh filename="package://kamuy2_description/meshes/back_left_link_foot.stl" scale="0.001 0.001 0.001"/>
@@ -206,10 +206,10 @@
 <link name="front_left_link_foot">
   <inertial>
-    <origin xyz="0 0 0" rpy="0 0 0"/>
+    <origin xyz="0 0 0" rpy="0 1.570796 0"/>
     <mass value="0.2932724386587248"/>
     <inertia ixx="0.002288" iyy="0.002324" izz="0.00015" ixy="4e-06" iyz="1e-05" ixz="-0.000187"/>
   </inertial>
   <visual>
-    <origin xyz="0 0 0" rpy="0 0 0"/>
+    <origin xyz="0 0 0" rpy="0 1.570796 0"/>
     <geometry>
       <mesh filename="package://kamuy2_description/meshes/front_left_link_foot.stl" scale="0.001 0.001 0.001"/>
@@ -218,5 +218,5 @@
   </visual>
   <collision>
-    <origin xyz="0 0 0" rpy="0 0 0"/>
+    <origin xyz="0 0 0" rpy="0 1.570796 0"/>
     <geometry>
       <mesh filename="package://kamuy2_description/meshes/front_left_link_foot.stl" scale="0.001 0.001 0.001"/>
@@ -226,10 +226,10 @@
 <link name="front_right_link_foot">
   <inertial>
-    <origin xyz="0 0 0" rpy="3.141592 0 0"/>
+    <origin xyz="0 0 0" rpy="3.141592 1.570796 0"/>
     <mass value="0.29327243865872493"/>
     <inertia ixx="0.002288" iyy="0.002324" izz="0.00015" ixy="-4e-06" iyz="-1e-05" ixz="-0.000187"/>
   </inertial>
   <visual>
-    <origin xyz="0 0 0" rpy="3.141592 0 0"/>
+    <origin xyz="0 0 0" rpy="3.141592 1.570796 0"/>
     <geometry>
       <mesh filename="package://kamuy2_description/meshes/front_right_link_foot.stl" scale="0.001 0.001 0.001"/>
@@ -238,5 +238,5 @@
   </visual>
   <collision>
-    <origin xyz="0 0 0" rpy="3.141592 0 0"/>
+    <origin xyz="0 0 0" rpy="3.141592 1.570796 0"/>
     <geometry>
       <mesh filename="package://kamuy2_description/meshes/front_right_link_foot.stl" scale="0.001 0.001 0.001"/>
@@ -246,10 +246,10 @@
 <link name="back_right_link_foot">
   <inertial>
-    <origin xyz="0 0 0" rpy="3.141592 0 0"/>
+    <origin xyz="0 0 0" rpy="3.141592 1.570796 0"/>
     <mass value="0.29327243865872493"/>
     <inertia ixx="0.002288" iyy="0.002324" izz="0.00015" ixy="-4e-06" iyz="-1e-05" ixz="-0.000187"/>
   </inertial>
   <visual>
-    <origin xyz="0 0 0" rpy="3.141592 0 0"/>
+    <origin xyz="0 0 0" rpy="3.141592 1.570796 0"/>
     <geometry>
       <mesh filename="package://kamuy2_description/meshes/back_right_link_foot.stl" scale="0.001 0.001 0.001"/>
@@ -258,9 +258,17 @@
   </visual>
   <collision>
-    <origin xyz="0 0 0" rpy="3.141592 0 0"/>
+    <origin xyz="0 0 0" rpy="3.141592 1.570796 0"/>
     <geometry>
       <mesh filename="package://kamuy2_description/meshes/back_right_link_foot.stl" scale="0.001 0.001 0.001"/>
     </geometry>
   </collision>
+</link>
+<link name="front_left_foot">
+</link>
+<link name="front_right_foot">
+</link>
+<link name="back_left_foot">
+</link>
+<link name="back_right_foot">
 </link>
 <!--
@@ -389,6 +397,6 @@
   <parent link="back_left_link_first"/>
   <child link="back_left_link_second"/>
-  <axis xyz="-5e-06 -1.0 -0.0"/>
-  <limit upper="0.087266" lower="-3.141593" effort="100" velocity="100"/>
+  <axis xyz="0.0 1.0 0.0"/>
+  <limit upper="3.141593" lower="0.0" effort="100" velocity="100"/>
 </joint>
 <joint name="fr2" type="revolute">
@@ -403,33 +411,61 @@
   <parent link="back_right_link_first"/>
   <child link="back_right_link_second"/>
-  <axis xyz="-5e-06 -1.0 -0.0"/>
-  <limit upper="0.0" lower="-3.141593" effort="100" velocity="100"/>
+  <axis xyz="-0.0 1.0 -0.0"/>
+  <limit upper="3.141593" lower="0.0" effort="100" velocity="100"/>
 </joint>
 <joint name="bl3" type="revolute">
-  <origin xyz="0.200 0 0 " rpy="0 0 0"/>
+  <origin xyz=" 0 0 -0.200" rpy="0 0 0"/>
   <parent link="back_left_link_second"/>
   <child link="back_left_link_foot"/>
-  <axis xyz="-5e-06 -1.0 -0.0"/>
+  <axis xyz="0 1 -0.0"/>
   <limit upper="3.141593" lower="0.0" effort="100" velocity="100"/>
 </joint>
 <joint name="fl3" type="revolute">
-  <origin xyz="0.200 0 0" rpy="0 0 0"/>
+  <origin xyz="0 0 -0.200 " rpy="0 0 0"/>
   <parent link="front_left_link_second"/>
   <child link="front_left_link_foot"/>
-  <axis xyz="-0.0 -1.0 -0.0"/>
+  <axis xyz="-0.0 1.0 -0.0"/>
   <limit upper="3.141593" lower="0.0" effort="100" velocity="100"/>
 </joint>
 <joint name="fr3" type="revolute">
-  <origin xyz="0.200 0 0" rpy="0 0 0"/>
+  <origin xyz="0 0 -0.200 " rpy="0 0 0"/>
   <parent link="front_right_link_second"/>
   <child link="front_right_link_foot"/>
-  <axis xyz="0.0 -1.0 0.0"/>
+  <axis xyz="0.0 1.0 0.0"/>
   <limit upper="3.141593" lower="0.0" effort="100" velocity="100"/>
 </joint>
 <joint name="br3" type="revolute">
-  <origin xyz="0.200 0 0" rpy="0 0 0"/>
+  <origin xyz="0 0 -0.200 " rpy="0 0 0"/>
   <parent link="back_right_link_second"/>
   <child link="back_right_link_foot"/>
-  <axis xyz="-5e-06 -1.0 -0.0"/>
+  <axis xyz="0 1.0 -0.0"/>
+  <limit upper="3.141593" lower="0.0" effort="100" velocity="100"/>
+</joint>
+<joint name="fl4" type="fixed">
+  <origin xyz="-0.05 0 -0.22" rpy="0 0 0"/>
+  <parent link="front_left_link_foot"/>
+  <child link="front_left_foot"/>
+  <axis xyz="0.0 1.0 -0.0"/>
+  <limit upper="3.141593" lower="0.0" effort="100" velocity="100"/>
+</joint>
+<joint name="fr4" type="fixed">
+ <origin xyz="-0.05 0 -0.22 " rpy="0 0 0"/>
+  <parent link="front_right_link_foot"/>
+  <child link="front_right_foot"/>
+  <axis xyz="0.0 1.0 -0.0"/>
+  <limit upper="3.141593" lower="0.0" effort="100" velocity="100"/>
+</joint>
+<joint name="bl4" type="fixed">
+  <origin xyz="-0.05 0 -0.22" rpy="0 0 0"/>
+  <parent link="back_left_link_foot"/>
+  <child link="back_left_foot"/>
+  <axis xyz="0.0 1.0 -0.0"/>
+  <limit upper="3.141593" lower="0.0" effort="100" velocity="100"/>
+</joint>
+<joint name="br4" type="fixed">
+ <origin xyz="-0.05 0 -0.22" rpy="0 0 0"/>
+  <parent link="back_right_link_foot"/>
+  <child link="back_right_foot"/>
+  <axis xyz="-0.0 -1.0 -0.0"/>
   <limit upper="3.141593" lower="0.0" effort="100" velocity="100"/>
 </joint>

Commit message: realsense

File: urdf/kamuy2.xacro (robot description, xacro)
@@ -4,4 +4,5 @@
 <xacro:include filename="$(find kamuy2_description)/urdf/kamuy2.trans" />
 <xacro:include filename="$(find kamuy2_description)/urdf/kamuy2.gazebo" />
+<xacro:include filename="$(find realsense2_description)/urdf/_d435.urdf.xacro"/>
 <link name="base_link">
   <inertial>
@@ -33,13 +34,7 @@
 </link>
 <!-- sensor -->
-<link name="camera_link">
-  <visual>
-    <origin xyz="0 0.0 0" rpy="0 0 0"/>
-    <geometry>
-      <sphere radius="0.05"/>
-    </geometry>
-    <material name="silver"/>
-  </visual>
-</link>
+<xacro:sensor_d435 name="camera" parent="base_link" publish_pointcloud="true">
+    <origin xyz="0.307 0 0.1" rpy="0 0.392699 0" />
+</xacro:sensor_d435>
 <link name="imu_link">
   <visual>
@@ -697,10 +692,10 @@
   <limit upper="3.141593" lower="0.0" effort="20" velocity="1.5"/>
 </joint>
-<joint name="camera_joint" type="fixed">
+<!-- <joint name="camera_joint" type="fixed">
  <origin xyz="0.3 0 0" rpy="0 0 0"/>
   <parent link="base_link"/>
   <child link="camera_link"/>
   <axis xyz="0 0 0"/>
-</joint>
+</joint> -->
 <joint name="imu_joint" type="fixed">
  <origin xyz="0 0 0" rpy="0 0 0"/>

File: urdf/kamuy2_champ.urdf (robot description, URDF)
Before this commit: robot kamuy2, 20 links, 19 joints
Links:
- added link camera_bottom_screw_frame
- added link camera_color_frame
- added link camera_color_optical_frame
- added link camera_depth_frame
- added link camera_depth_optical_frame
- added link camera_left_ir_frame
- added link camera_left_ir_optical_frame
- added link camera_right_ir_frame
- added link camera_right_ir_optical_frame
- link camera_link: mass None -> 0.564; geometry collision box size=0.02505 0.09 0.025; visual mesh filename=package://realsense2_description/meshes/d435.dae
Joints:
- added joint camera_color_joint: type fixed, parent camera_depth_frame, child camera_color_frame, origin xyz=0 0.015 0 rpy=0 0 0
- added joint camera_color_optical_joint: type fixed, parent camera_color_frame, child camera_color_optical_frame, origin xyz=0 0 0 rpy=-1.5707963267948966 0 -1.5707963267948966
- added joint camera_depth_joint: type fixed, parent camera_link, child camera_depth_frame, origin xyz=0 0 0 rpy=0 0 0
- added joint camera_depth_optical_joint: type fixed, parent camera_depth_frame, child camera_depth_optical_frame, origin xyz=0 0 0 rpy=-1.5707963267948966 0 -1.5707963267948966
- added joint camera_left_ir_joint: type fixed, parent camera_depth_frame, child camera_left_ir_frame, origin xyz=0 0.0 0 rpy=0 0 0
- added joint camera_left_ir_optical_joint: type fixed, parent camera_left_ir_frame, child camera_left_ir_optical_frame, origin xyz=0 0 0 rpy=-1.5707963267948966 0 -1.5707963267948966
- added joint camera_link_joint: type fixed, parent camera_bottom_screw_frame, child camera_link, origin xyz=0 0.0175 0.0125 rpy=0 0 0
- added joint camera_right_ir_joint: type fixed, parent camera_depth_frame, child camera_right_ir_frame, origin xyz=0 -0.05 0 rpy=0 0 0
- added joint camera_right_ir_optical_joint: type fixed, parent camera_right_ir_frame, child camera_right_ir_optical_frame, origin xyz=0 0 0 rpy=-1.5707963267948966 0 -1.5707963267948966
- joint camera_joint: axis 0 0 0 -> (none); child camera_link -> camera_bottom_screw_frame; origin xyz=0.3 0 0 rpy=0 0 0 -> xyz=0.307 0 0.1 rpy=0 0.392699 0
